File: lab4/lab4 exercise1/lab4.kicad_sch (KiCad schematic)
At the start: 6 parts, among them SW1 s

Commit message: updated lab4 from lab6 instructions
Parts:
- C1: footprint (none) -> Capacitor_THT:C_Radial_D5.0mm_H5.0mm_P2.00mm
- D1: footprint (none) -> LED_THT:LED_D5.0mm
- R1, R2: footprint (none) -> Resistor_THT:R_Axial_DIN0516_L15.5mm_D5.0mm_P20.32mm_Horizontal
- SW1: footprint (none) -> Button_Switch_THT:SW_E-Switch_EG1224_SPDT_Angled
- V1: footprint (none) -> Connector_JST:JST_PH_B2B-PH-K_1x02_P2.00mm_Vertical
Changed lines of the file:
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@@
       (effects (font (size 1.27 1.27)) (justify left))
     )
-    (property "Footprint" "" (id 2) (at 177.8 92.71 90)
+    (property "Footprint" "LED_THT:LED_D5.0mm" (id 2) (at 177.8 92.71 90)
       (effects (font (size 1.27 1.27)) hide)
     )
@@
       (effects (font (size 1.27 1.27)) hide)
     )
-    (property "Footprint" "" (id 2) (at 133.35 67.31 0)
+    (property "Footprint" "Button_Switch_THT:SW_E-Switch_EG1224_SPDT_Angled" (id 2) (at 133.35 67.31 0)
       (effects (font (size 1.27 1.27)) hide)
     )
@@
     (property "Reference" "V1" (id 0) (at 105.41 87.63 0))
     (property "Value" "9V" (id 1) (at 105.41 90.17 0))
-    (property "Footprint" "" (id 2) (at 96.52 87.63 0)
+    (property "Footprint" "Connector_JST:JST_PH_B2B-PH-K_1x02_P2.00mm_Vertical" (id 2) (at 96.52 87.63 0)
       (effects (font (size 1.27 1.27)) hide)
     )
@@
       (effects (font (size 1.27 1.27)) (justify left))
     )
-    (property "Footprint" "" (id 2) (at 144.4752 91.44 0)
+    (property "Footprint" "Capacitor_THT:C_Radial_D5.0mm_H5.0mm_P2.00mm" (id 2) (at 144.4752 91.44 0)
       (effects (font (size 1.27 1.27)) hide)
     )
@@
     (property "Reference" "R2" (id 0) (at 116.84 69.85 0))
     (property "Value" "2.2 kΩ" (id 1) (at 116.84 72.39 0))
-    (property "Footprint" "" (id 2) (at 113.792 68.58 90)
+    (property "Footprint" "Resistor_THT:R_Axial_DIN0516_L15.5mm_D5.0mm_P20.32mm_Horizontal" (id 2) (at 113.792 68.58 90)
       (effects (font (size 1.27 1.27)) hide)
     )
@@
       (effects (font (size 1.27 1.27)) (justify left))
     )
-    (property "Footprint" "" (id 2) (at 179.07 81.788 0)
+    (property "Footprint" "Resistor_THT:R_Axial_DIN0516_L15.5mm_D5.0mm_P20.32mm_Horizontal" (id 2) (at 179.07 81.788 0)
       (effects (font (size 1.27 1.27)) hide)
     )
@@
   (symbol_instances
     (path "/55b7af21-7f4e-480f-863d-7dbdbf25334a"
-      (reference "C1") (unit 1) (value "4.7 µF") (footprint "")
+      (reference "C1") (unit 1) (value "4.7 µF") (footprint "Capacitor_THT:C_Radial_D5.0mm_H5.0mm_P2.00mm")
     )
     (path "/11b344e8-3c8e-47cd-8c60-bff25554c3d0"
-      (reference "D1") (unit 1) (value "LED") (footprint "")
+      (reference "D1") (unit 1) (value "LED") (footprint "LED_THT:LED_D5.0mm")
     )
     (path "/e06620fc-ae98-4314-818e-b4f8152b7fd2"
-      (reference "R1") (unit 1) (value "20 kΩ") (footprint "")
+      (reference "R1") (unit 1) (value "20 kΩ") (footprint "Resistor_THT:R_Axial_DIN0516_L15.5mm_D5.0mm_P20.32mm_Horizontal")
     )
     (path "/8b92f818-8b21-4c79-84ca-80ea4e9c1810"
-      (reference "R2") (unit 1) (value "2.2 kΩ") (footprint "")
+      (reference "R2") (unit 1) (value "2.2 kΩ") (footprint "Resistor_THT:R_Axial_DIN0516_L15.5mm_D5.0mm_P20.32mm_Horizontal")
     )
     (path "/2ce80727-87c9-4db6-94e2-c63b4538046f"
-      (reference "SW1") (unit 1) (value "s") (footprint "")
+      (reference "SW1") (unit 1) (value "s") (footprint "Button_Switch_THT:SW_E-Switch_EG1224_SPDT_Angled")
     )
     (path "/37a44659-0373-4363-9c08-7156d0e7a677"
-      (reference "V1") (unit 1) (value "9V") (footprint "")
+      (reference "V1") (unit 1) (value "9V") (footprint "Connector_JST:JST_PH_B2B-PH-K_1x02_P2.00mm_Vertical")
     )
   )
